Commit message: generated arm files

File: urdf/arm.xacro (robot description, xacro)
@@ -23,19 +23,19 @@
             <geometry>
                 <mesh
-                    filename="package://mirte_master_description/meshes/arm_Rot.STL" />
-            </geometry>
-            <material
-                name="">
-                <color
-                    rgba="0.792156862745098 0.819607843137255 0.933333333333333 1" />
-            </material>
-        </visual>
-        <collision>
-            <origin
-                xyz="0 0 0"
-                rpy="0 0 0" />
-            <geometry>
-                <mesh
-                    filename="package://mirte_master_description/meshes/arm_Rot.STL" />
+                    filename="package://mirte_arm_description/meshes/arm_Rot.STL" />
+            </geometry>
+            <material
+                name="">
+                <color
+                    rgba="0.792156862745098 0.819607843137255 0.933333333333333 1" />
+            </material>
+        </visual>
+        <collision>
+            <origin
+                xyz="0 0 0"
+                rpy="0 0 0" />
+            <geometry>
+                <mesh
+                    filename="package://mirte_arm_description/meshes/arm_Rot.STL" />
             </geometry>
         </collision>
@@ -82,5 +82,5 @@
             <geometry>
                 <mesh
-                    filename="package://mirte_master_description/meshes/arm_Shoulder.STL" />
+                    filename="package://mirte_arm_description/meshes/arm_Shoulder.STL" />
             </geometry>
             <material
@@ -96,5 +96,5 @@
             <geometry>
                 <mesh
-                    filename="package://mirte_master_description/meshes/arm_Shoulder.STL" />
+                    filename="package://mirte_arm_description/meshes/arm_Shoulder.STL" />
             </geometry>
         </collision>
@@ -141,5 +141,5 @@
             <geometry>
                 <mesh
-                    filename="package://mirte_master_description/meshes/arm_Elbow.STL" />
+                    filename="package://mirte_arm_description/meshes/arm_Elbow.STL" />
             </geometry>
             <material
@@ -155,5 +155,5 @@
             <geometry>
                 <mesh
-                    filename="package://mirte_master_description/meshes/arm_Elbow.STL" />
+                    filename="package://mirte_arm_description/meshes/arm_Elbow.STL" />
             </geometry>
         </collision>
@@ -200,5 +200,5 @@
             <geometry>
                 <mesh
-                    filename="package://mirte_master_description/meshes/arm_Wrist.STL" />
+                    filename="package://mirte_arm_description/meshes/arm_Wrist.STL" />
             </geometry>
             <material
@@ -214,5 +214,5 @@
             <geometry>
                 <mesh
-                    filename="package://mirte_master_description/meshes/arm_Wrist.STL" />
+                    filename="package://mirte_arm_description/meshes/arm_Wrist.STL" />
             </geometry>
         </collision>
@@ -259,19 +259,19 @@
             <geometry>
                 <mesh
-                    filename="package://mirte_master_description/meshes/Gripper.STL" />
-            </geometry>
-            <material
-                name="">
-                <color
-                    rgba="0.792156862745098 0.819607843137255 0.933333333333333 1" />
-            </material>
-        </visual>
-        <collision>
-            <origin
-                xyz="0 0 0"
-                rpy="0 0 0" />
-            <geometry>
-                <mesh
-                    filename="package://mirte_master_description/meshes/Gripper.STL" />
+                    filename="package://mirte_arm_description/meshes/Gripper.STL" />
+            </geometry>
+            <material
+                name="">
+                <color
+                    rgba="0.792156862745098 0.819607843137255 0.933333333333333 1" />
+            </material>
+        </visual>
+        <collision>
+            <origin
+                xyz="0 0 0"
+                rpy="0 0 0" />
+            <geometry>
+                <mesh
+                    filename="package://mirte_arm_description/meshes/Gripper.STL" />
             </geometry>
         </collision>
@@ -318,19 +318,19 @@
             <geometry>
                 <mesh
-                    filename="package://mirte_master_description/meshes/_gripper_link_r.STL" />
-            </geometry>
-            <material
-                name="">
-                <color
-                    rgba="0.792156862745098 0.819607843137255 0.933333333333333 1" />
-            </material>
-        </visual>
-        <collision>
-            <origin
-                xyz="0 0 0"
-                rpy="0 0 0" />
-            <geometry>
-                <mesh
-                    filename="package://mirte_master_description/meshes/_gripper_link_r.STL" />
+                    filename="package://mirte_arm_description/meshes/_gripper_link_r.STL" />
+            </geometry>
+            <material
+                name="">
+                <color
+                    rgba="0.792156862745098 0.819607843137255 0.933333333333333 1" />
+            </material>
+        </visual>
+        <collision>
+            <origin
+                xyz="0 0 0"
+                rpy="0 0 0" />
+            <geometry>
+                <mesh
+                    filename="package://mirte_arm_description/meshes/_gripper_link_r.STL" />
             </geometry>
         </collision>
@@ -376,19 +376,19 @@
             <geometry>
                 <mesh
-                    filename="package://mirte_master_description/meshes/gripper_finger_r.STL" />
-            </geometry>
-            <material
-                name="">
-                <color
-                    rgba="0.792156862745098 0.819607843137255 0.933333333333333 1" />
-            </material>
-        </visual>
-        <collision>
-            <origin
-                xyz="0 0 0"
-                rpy="0 0 0" />
-            <geometry>
-                <mesh
-                    filename="package://mirte_master_description/meshes/gripper_finger_r.STL" />
+                    filename="package://mirte_arm_description/meshes/gripper_finger_r.STL" />
+            </geometry>
+            <material
+                name="">
+                <color
+                    rgba="0.792156862745098 0.819607843137255 0.933333333333333 1" />
+            </material>
+        </visual>
+        <collision>
+            <origin
+                xyz="0 0 0"
+                rpy="0 0 0" />
+            <geometry>
+                <mesh
+                    filename="package://mirte_arm_description/meshes/gripper_finger_r.STL" />
             </geometry>
         </collision>
@@ -434,19 +434,19 @@
             <geometry>
                 <mesh
-                    filename="package://mirte_master_description/meshes/_gripper_link_l.STL" />
-            </geometry>
-            <material
-                name="">
-                <color
-                    rgba="0.792156862745098 0.819607843137255 0.933333333333333 1" />
-            </material>
-        </visual>
-        <collision>
-            <origin
-                xyz="0 0 0"
-                rpy="0 0 0" />
-            <geometry>
-                <mesh
-                    filename="package://mirte_master_description/meshes/_gripper_link_l.STL" />
+                    filename="package://mirte_arm_description/meshes/_gripper_link_l.STL" />
+            </geometry>
+            <material
+                name="">
+                <color
+                    rgba="0.792156862745098 0.819607843137255 0.933333333333333 1" />
+            </material>
+        </visual>
+        <collision>
+            <origin
+                xyz="0 0 0"
+                rpy="0 0 0" />
+            <geometry>
+                <mesh
+                    filename="package://mirte_arm_description/meshes/_gripper_link_l.STL" />
             </geometry>
         </collision>
@@ -492,19 +492,19 @@
             <geometry>
                 <mesh
-                    filename="package://mirte_master_description/meshes/gripper_finger_l.STL" />
-            </geometry>
-            <material
-                name="">
-                <color
-                    rgba="0.792156862745098 0.819607843137255 0.933333333333333 1" />
-            </material>
-        </visual>
-        <collision>
-            <origin
-                xyz="0 0 0"
-                rpy="0 0 0" />
-            <geometry>
-                <mesh
-                    filename="package://mirte_master_description/meshes/gripper_finger_l.STL" />
+                    filename="package://mirte_arm_description/meshes/gripper_finger_l.STL" />
+            </geometry>
+            <material
+                name="">
+                <color
+                    rgba="0.792156862745098 0.819607843137255 0.933333333333333 1" />
+            </material>
+        </visual>
+        <collision>
+            <origin
+                xyz="0 0 0"
+                rpy="0 0 0" />
+            <geometry>
+                <mesh
+                    filename="package://mirte_arm_description/meshes/gripper_finger_l.STL" />
             </geometry>
         </collision>
@@ -550,19 +550,19 @@
             <geometry>
                 <mesh
-                    filename="package://mirte_master_description/meshes/_Gripper_r.STL" />
-            </geometry>
-            <material
-                name="">
-                <color
-                    rgba="0.792156862745098 0.819607843137255 0.933333333333333 1" />
-            </material>
-        </visual>
-        <collision>
-            <origin
-                xyz="0 0 0"
-                rpy="0 0 0" />
-            <geometry>
-                <mesh
-                    filename="package://mirte_master_description/meshes/_Gripper_r.STL" />
+                    filename="package://mirte_arm_description/meshes/_Gripper_r.STL" />
+            </geometry>
+            <material
+                name="">
+                <color
+                    rgba="0.792156862745098 0.819607843137255 0.933333333333333 1" />
+            </material>
+        </visual>
+        <collision>
+            <origin
+                xyz="0 0 0"
+                rpy="0 0 0" />
+            <geometry>
+                <mesh
+                    filename="package://mirte_arm_description/meshes/_Gripper_r.STL" />
             </geometry>
         </collision>

Commit message: modified param filename

File: urdf/arm.xacro (robot description, xacro)
@@ -23,19 +23,19 @@
             <geometry>
                 <mesh
-                    filename="package://mirte_arm_description/meshes/arm_Rot.STL" />
-            </geometry>
-            <material
-                name="">
-                <color
-                    rgba="0.792156862745098 0.819607843137255 0.933333333333333 1" />
-            </material>
-        </visual>
-        <collision>
-            <origin
-                xyz="0 0 0"
-                rpy="0 0 0" />
-            <geometry>
-                <mesh
-                    filename="package://mirte_arm_description/meshes/arm_Rot.STL" />
+                    filename="package://mirte_master_description/meshes/arm_Rot.STL" />
+            </geometry>
+            <material
+                name="">
+                <color
+                    rgba="0.792156862745098 0.819607843137255 0.933333333333333 1" />
+            </material>
+        </visual>
+        <collision>
+            <origin
+                xyz="0 0 0"
+                rpy="0 0 0" />
+            <geometry>
+                <mesh
+                    filename="package://mirte_master_description/meshes/arm_Rot.STL" />
             </geometry>
         </collision>
@@ -82,5 +82,5 @@
             <geometry>
                 <mesh
-                    filename="package://mirte_arm_description/meshes/arm_Shoulder.STL" />
+                    filename="package://mirte_master_description/meshes/arm_Shoulder.STL" />
             </geometry>
             <material
@@ -96,5 +96,5 @@
             <geometry>
                 <mesh
-                    filename="package://mirte_arm_description/meshes/arm_Shoulder.STL" />
+                    filename="package://mirte_master_description/meshes/arm_Shoulder.STL" />
             </geometry>
         </collision>
@@ -141,5 +141,5 @@
             <geometry>
                 <mesh
-                    filename="package://mirte_arm_description/meshes/arm_Elbow.STL" />
+                    filename="package://mirte_master_description/meshes/arm_Elbow.STL" />
             </geometry>
             <material
@@ -155,5 +155,5 @@
             <geometry>
                 <mesh
-                    filename="package://mirte_arm_description/meshes/arm_Elbow.STL" />
+                    filename="package://mirte_master_description/meshes/arm_Elbow.STL" />
             </geometry>
         </collision>
@@ -200,5 +200,5 @@
             <geometry>
                 <mesh
-                    filename="package://mirte_arm_description/meshes/arm_Wrist.STL" />
+                    filename="package://mirte_master_description/meshes/arm_Wrist.STL" />
             </geometry>
             <material
@@ -214,5 +214,5 @@
             <geometry>
                 <mesh
-                    filename="package://mirte_arm_description/meshes/arm_Wrist.STL" />
+                    filename="package://mirte_master_description/meshes/arm_Wrist.STL" />
             </geometry>
         </collision>
@@ -259,19 +259,19 @@
             <geometry>
                 <mesh
-                    filename="package://mirte_arm_description/meshes/Gripper.STL" />
-            </geometry>
-            <material
-                name="">
-                <color
-                    rgba="0.792156862745098 0.819607843137255 0.933333333333333 1" />
-            </material>
-        </visual>
-        <collision>
-            <origin
-                xyz="0 0 0"
-                rpy="0 0 0" />
-            <geometry>
-                <mesh
-                    filename="package://mirte_arm_description/meshes/Gripper.STL" />
+                    filename="package://mirte_master_description/meshes/Gripper.STL" />
+            </geometry>
+            <material
+                name="">
+                <color
+                    rgba="0.792156862745098 0.819607843137255 0.933333333333333 1" />
+            </material>
+        </visual>
+        <collision>
+            <origin
+                xyz="0 0 0"
+                rpy="0 0 0" />
+            <geometry>
+                <mesh
+                    filename="package://mirte_master_description/meshes/Gripper.STL" />
             </geometry>
         </collision>
@@ -318,19 +318,19 @@
             <geometry>
                 <mesh
-                    filename="package://mirte_arm_description/meshes/_gripper_link_r.STL" />
-            </geometry>
-            <material
-                name="">
-                <color
-                    rgba="0.792156862745098 0.819607843137255 0.933333333333333 1" />
-            </material>
-        </visual>
-        <collision>
-            <origin
-                xyz="0 0 0"
-                rpy="0 0 0" />
-            <geometry>
-                <mesh
-                    filename="package://mirte_arm_description/meshes/_gripper_link_r.STL" />
+                    filename="package://mirte_master_description/meshes/_gripper_link_r.STL" />
+            </geometry>
+            <material
+                name="">
+                <color
+                    rgba="0.792156862745098 0.819607843137255 0.933333333333333 1" />
+            </material>
+        </visual>
+        <collision>
+            <origin
+                xyz="0 0 0"
+                rpy="0 0 0" />
+            <geometry>
+                <mesh
+                    filename="package://mirte_master_description/meshes/_gripper_link_r.STL" />
             </geometry>
         </collision>
@@ -376,19 +376,19 @@
             <geometry>
                 <mesh
-                    filename="package://mirte_arm_description/meshes/gripper_finger_r.STL" />
-            </geometry>
-            <material
-                name="">
-                <color
-                    rgba="0.792156862745098 0.819607843137255 0.933333333333333 1" />
-            </material>
-        </visual>
-        <collision>
-            <origin
-                xyz="0 0 0"
-                rpy="0 0 0" />
-            <geometry>
-                <mesh
-                    filename="package://mirte_arm_description/meshes/gripper_finger_r.STL" />
+                    filename="package://mirte_master_description/meshes/gripper_finger_r.STL" />
+            </geometry>
+            <material
+                name="">
+                <color
+                    rgba="0.792156862745098 0.819607843137255 0.933333333333333 1" />
+            </material>
+        </visual>
+        <collision>
+            <origin
+                xyz="0 0 0"
+                rpy="0 0 0" />
+            <geometry>
+                <mesh
+                    filename="package://mirte_master_description/meshes/gripper_finger_r.STL" />
             </geometry>
         </collision>
@@ -434,19 +434,19 @@
             <geometry>
                 <mesh
-                    filename="package://mirte_arm_description/meshes/_gripper_link_l.STL" />
-            </geometry>
-            <material
-                name="">
-                <color
-                    rgba="0.792156862745098 0.819607843137255 0.933333333333333 1" />
-            </material>
-        </visual>
-        <collision>
-            <origin
-                xyz="0 0 0"
-                rpy="0 0 0" />
-            <geometry>
-                <mesh
-                    filename="package://mirte_arm_description/meshes/_gripper_link_l.STL" />
+                    filename="package://mirte_master_description/meshes/_gripper_link_l.STL" />
+            </geometry>
+            <material
+                name="">
+                <color
+                    rgba="0.792156862745098 0.819607843137255 0.933333333333333 1" />
+            </material>
+        </visual>
+        <collision>
+            <origin
+                xyz="0 0 0"
+                rpy="0 0 0" />
+            <geometry>
+                <mesh
+                    filename="package://mirte_master_description/meshes/_gripper_link_l.STL" />
             </geometry>
         </collision>
@@ -492,19 +492,19 @@
             <geometry>
                 <mesh
-                    filename="package://mirte_arm_description/meshes/gripper_finger_l.STL" />
-            </geometry>
-            <material
-                name="">
-                <color
-                    rgba="0.792156862745098 0.819607843137255 0.933333333333333 1" />
-            </material>
-        </visual>
-        <collision>
-            <origin
-                xyz="0 0 0"
-                rpy="0 0 0" />
-            <geometry>
-                <mesh
-                    filename="package://mirte_arm_description/meshes/gripper_finger_l.STL" />
+                    filename="package://mirte_master_description/meshes/gripper_finger_l.STL" />
+            </geometry>
+            <material
+                name="">
+                <color
+                    rgba="0.792156862745098 0.819607843137255 0.933333333333333 1" />
+            </material>
+        </visual>
+        <collision>
+            <origin
+                xyz="0 0 0"
+                rpy="0 0 0" />
+            <geometry>
+                <mesh
+                    filename="package://mirte_master_description/meshes/gripper_finger_l.STL" />
             </geometry>
         </collision>
@@ -550,19 +550,19 @@
             <geometry>
                 <mesh
-                    filename="package://mirte_arm_description/meshes/_Gripper_r.STL" />
-            </geometry>
-            <material
-                name="">
-                <color
-                    rgba="0.792156862745098 0.819607843137255 0.933333333333333 1" />
-            </material>
-        </visual>
-        <collision>
-            <origin
-                xyz="0 0 0"
-                rpy="0 0 0" />
-            <geometry>
-                <mesh
-                    filename="package://mirte_arm_description/meshes/_Gripper_r.STL" />
+                    filename="package://mirte_master_description/meshes/_Gripper_r.STL" />
+            </geometry>
+            <material
+                name="">
+                <color
+                    rgba="0.792156862745098 0.819607843137255 0.933333333333333 1" />
+            </material>
+        </visual>
+        <collision>
+            <origin
+                xyz="0 0 0"
+                rpy="0 0 0" />
+            <geometry>
+                <mesh
+                    filename="package://mirte_master_description/meshes/_Gripper_r.STL" />
             </geometry>
         </collision>
