Commit message: fixed the xacro file. added a urdf

File: urdf/arm.xacro (robot description, xacro)
@@ -1,4 +1,10 @@
 <?xml version="1.0" encoding="UTF-8"?>
-<robot xmlns:xacro="http://www.ros.org/wiki/xacro">
+<!-- This URDF was automatically created by SolidWorks to URDF Exporter! Originally created by
+Stephen Brawner (brawner@gmail.com)
+     Commit Version: 1.6.0-4-g7f85cfe  Build Version: 1.6.7995.38578
+     For more information, please see http://wiki.ros.org/sw_urdf_exporter -->
+<robot
+  name="mirte_master" xmlns:xacro="http://ros.org/wiki/xacro">
+    <link name="base_link" />
     <link
         name="arm_Rot">
@@ -23,19 +29,19 @@
             <geometry>
                 <mesh
-                    filename="package://mirte_master_description/meshes/arm_Rot.STL" />
-            </geometry>
-            <material
-                name="">
-                <color
-                    rgba="0.792156862745098 0.819607843137255 0.933333333333333 1" />
-            </material>
-        </visual>
-        <collision>
-            <origin
-                xyz="0 0 0"
-                rpy="0 0 0" />
-            <geometry>
-                <mesh
-                    filename="package://mirte_master_description/meshes/arm_Rot.STL" />
+                    filename="package://mirte_arm_description/meshes/arm_Rot.STL" />
+            </geometry>
+            <material
+                name="">
+                <color
+                    rgba="0.792156862745098 0.819607843137255 0.933333333333333 1" />
+            </material>
+        </visual>
+        <collision>
+            <origin
+                xyz="0 0 0"
+                rpy="0 0 0" />
+            <geometry>
+                <mesh
+                    filename="package://mirte_arm_description/meshes/arm_Rot.STL" />
             </geometry>
         </collision>
@@ -48,5 +54,5 @@
             rpy="1.5708 0 3.1416" />
         <parent
-            link="frame_link" />
+            link="base_link" />
         <child
             link="arm_Rot" />
@@ -54,6 +60,6 @@
             xyz="0 1 0" />
         <limit
-            lower="${pi/-2}"
-            upper="${pi/2}"
+            lower="-1.5707"
+            upper="1.5707"
             effort="2"
             velocity="2"
@@ -82,5 +88,5 @@
             <geometry>
                 <mesh
-                    filename="package://mirte_master_description/meshes/arm_Shoulder.STL" />
+                    filename="package://mirte_arm_description/meshes/arm_Shoulder.STL" />
             </geometry>
             <material
@@ -96,5 +102,5 @@
             <geometry>
                 <mesh
-                    filename="package://mirte_master_description/meshes/arm_Shoulder.STL" />
+                    filename="package://mirte_arm_description/meshes/arm_Shoulder.STL" />
             </geometry>
         </collision>
@@ -113,6 +119,6 @@
             xyz="0 1 0" />
         <limit
-            lower="${pi/-2}"
-            upper="${pi/2}"
+            lower="-1.5707"
+            upper="1.5707"
             effort="2"
             velocity="2"
@@ -141,5 +147,5 @@
             <geometry>
                 <mesh
-                    filename="package://mirte_master_description/meshes/arm_Elbow.STL" />
+                    filename="package://mirte_arm_description/meshes/arm_Elbow.STL" />
             </geometry>
             <material
@@ -155,5 +161,5 @@
             <geometry>
                 <mesh
-                    filename="package://mirte_master_description/meshes/arm_Elbow.STL" />
+                    filename="package://mirte_arm_description/meshes/arm_Elbow.STL" />
             </geometry>
         </collision>
@@ -172,6 +178,6 @@
             xyz="1 0 0" />
         <limit
-            lower="${pi/-2}"
-            upper="${pi/2}"
+            lower="-1.5707"
+            upper="1.5707"
             effort="2"
             velocity="2"
@@ -200,5 +206,5 @@
             <geometry>
                 <mesh
-                    filename="package://mirte_master_description/meshes/arm_Wrist.STL" />
+                    filename="package://mirte_arm_description/meshes/arm_Wrist.STL" />
             </geometry>
             <material
@@ -214,5 +220,5 @@
             <geometry>
                 <mesh
-                    filename="package://mirte_master_description/meshes/arm_Wrist.STL" />
+                    filename="package://mirte_arm_description/meshes/arm_Wrist.STL" />
             </geometry>
         </collision>
@@ -231,6 +237,6 @@
             xyz="0 1 0" />
         <limit
-            lower="${pi/-2}"
-            upper="${pi/2}"
+            lower="-1.5707"
+            upper="1.5707"
             effort="2"
             velocity="2"
@@ -259,19 +265,19 @@
             <geometry>
                 <mesh
-                    filename="package://mirte_master_description/meshes/Gripper.STL" />
-            </geometry>
-            <material
-                name="">
-                <color
-                    rgba="0.792156862745098 0.819607843137255 0.933333333333333 1" />
-            </material>
-        </visual>
-        <collision>
-            <origin
-                xyz="0 0 0"
-                rpy="0 0 0" />
-            <geometry>
-                <mesh
-                    filename="package://mirte_master_description/meshes/Gripper.STL" />
+                    filename="package://mirte_arm_description/meshes/Gripper.STL" />
+            </geometry>
+            <material
+                name="">
+                <color
+                    rgba="0.792156862745098 0.819607843137255 0.933333333333333 1" />
+            </material>
+        </visual>
+        <collision>
+            <origin
+                xyz="0 0 0"
+                rpy="0 0 0" />
+            <geometry>
+                <mesh
+                    filename="package://mirte_arm_description/meshes/Gripper.STL" />
             </geometry>
         </collision>
@@ -291,5 +297,5 @@
         <limit
             lower="0"
-            upper="${pi/2}"
+            upper="1.5707"
             effort="2"
             velocity="2"
@@ -318,19 +324,19 @@
             <geometry>
                 <mesh
-                    filename="package://mirte_master_description/meshes/_gripper_link_r.STL" />
-            </geometry>
-            <material
-                name="">
-                <color
-                    rgba="0.792156862745098 0.819607843137255 0.933333333333333 1" />
-            </material>
-        </visual>
-        <collision>
-            <origin
-                xyz="0 0 0"
-                rpy="0 0 0" />
-            <geometry>
-                <mesh
-                    filename="package://mirte_master_description/meshes/_gripper_link_r.STL" />
+                    filename="package://mirte_arm_description/meshes/_gripper_link_r.STL" />
+            </geometry>
+            <material
+                name="">
+                <color
+                    rgba="0.792156862745098 0.819607843137255 0.933333333333333 1" />
+            </material>
+        </visual>
+        <collision>
+            <origin
+                xyz="0 0 0"
+                rpy="0 0 0" />
+            <geometry>
+                <mesh
+                    filename="package://mirte_arm_description/meshes/_gripper_link_r.STL" />
             </geometry>
         </collision>
@@ -376,19 +382,19 @@
             <geometry>
                 <mesh
-                    filename="package://mirte_master_description/meshes/gripper_finger_r.STL" />
-            </geometry>
-            <material
-                name="">
-                <color
-                    rgba="0.792156862745098 0.819607843137255 0.933333333333333 1" />
-            </material>
-        </visual>
-        <collision>
-            <origin
-                xyz="0 0 0"
-                rpy="0 0 0" />
-            <geometry>
-                <mesh
-                    filename="package://mirte_master_description/meshes/gripper_finger_r.STL" />
+                    filename="package://mirte_arm_description/meshes/gripper_finger_r.STL" />
+            </geometry>
+            <material
+                name="">
+                <color
+                    rgba="0.792156862745098 0.819607843137255 0.933333333333333 1" />
+            </material>
+        </visual>
+        <collision>
+            <origin
+                xyz="0 0 0"
+                rpy="0 0 0" />
+            <geometry>
+                <mesh
+                    filename="package://mirte_arm_description/meshes/gripper_finger_r.STL" />
             </geometry>
         </collision>
@@ -434,19 +440,19 @@
             <geometry>
                 <mesh
-                    filename="package://mirte_master_description/meshes/_gripper_link_l.STL" />
-            </geometry>
-            <material
-                name="">
-                <color
-                    rgba="0.792156862745098 0.819607843137255 0.933333333333333 1" />
-            </material>
-        </visual>
-        <collision>
-            <origin
-                xyz="0 0 0"
-                rpy="0 0 0" />
-            <geometry>
-                <mesh
-                    filename="package://mirte_master_description/meshes/_gripper_link_l.STL" />
+                    filename="package://mirte_arm_description/meshes/_gripper_link_l.STL" />
+            </geometry>
+            <material
+                name="">
+                <color
+                    rgba="0.792156862745098 0.819607843137255 0.933333333333333 1" />
+            </material>
+        </visual>
+        <collision>
+            <origin
+                xyz="0 0 0"
+                rpy="0 0 0" />
+            <geometry>
+                <mesh
+                    filename="package://mirte_arm_description/meshes/_gripper_link_l.STL" />
             </geometry>
         </collision>
@@ -492,19 +498,19 @@
             <geometry>
                 <mesh
-                    filename="package://mirte_master_description/meshes/gripper_finger_l.STL" />
-            </geometry>
-            <material
-                name="">
-                <color
-                    rgba="0.792156862745098 0.819607843137255 0.933333333333333 1" />
-            </material>
-        </visual>
-        <collision>
-            <origin
-                xyz="0 0 0"
-                rpy="0 0 0" />
-            <geometry>
-                <mesh
-                    filename="package://mirte_master_description/meshes/gripper_finger_l.STL" />
+                    filename="package://mirte_arm_description/meshes/gripper_finger_l.STL" />
+            </geometry>
+            <material
+                name="">
+                <color
+                    rgba="0.792156862745098 0.819607843137255 0.933333333333333 1" />
+            </material>
+        </visual>
+        <collision>
+            <origin
+                xyz="0 0 0"
+                rpy="0 0 0" />
+            <geometry>
+                <mesh
+                    filename="package://mirte_arm_description/meshes/gripper_finger_l.STL" />
             </geometry>
         </collision>
@@ -550,19 +556,19 @@
             <geometry>
                 <mesh
-                    filename="package://mirte_master_description/meshes/_Gripper_r.STL" />
-            </geometry>
-            <material
-                name="">
-                <color
-                    rgba="0.792156862745098 0.819607843137255 0.933333333333333 1" />
-            </material>
-        </visual>
-        <collision>
-            <origin
-                xyz="0 0 0"
-                rpy="0 0 0" />
-            <geometry>
-                <mesh
-                    filename="package://mirte_master_description/meshes/_Gripper_r.STL" />
+                    filename="package://mirte_arm_description/meshes/_Gripper_r.STL" />
+            </geometry>
+            <material
+                name="">
+                <color
+                    rgba="0.792156862745098 0.819607843137255 0.933333333333333 1" />
+            </material>
+        </visual>
+        <collision>
+            <origin
+                xyz="0 0 0"
+                rpy="0 0 0" />
+            <geometry>
+                <mesh
+                    filename="package://mirte_arm_description/meshes/_Gripper_r.STL" />
             </geometry>
         </collision>
